File: electrical/hot-wand-lite.sch (EAGLE design)
At the start: 107 parts, among them IC1 12V R-78K12-2.0, IC2 AMS1117-5.0, Q1 NCHAN, Q2 SIS862ADN-T1-GE3, Q3 SIS862ADN-T1-GE3, Q4 DMTH64M2LPDWQ-13, Q5 SIS862ADN-T1-GE3, Q6 2N7002K, Q7 G3404, SW1 SWITCH-SPDT-2MNT-SLW-864574-5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, U1 SEEED-XIAO-SAMD21-TH-LOCKING, U2 1EDN8511BXUSA1, U3 LM74810QDRRRQ1, U4 AP53781

Commit message: Update hot-wand-lite.sch
Other:
- note removed: "mess with these resistors if LEDs are too dim"
Changed lines of the file:
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@@
 <text x="199.644" y="-621.284" size="1.778" layer="97" rot="R270" align="bottom-right">select 28V
 (26K eqv)</text>
-<text x="185.42" y="-312.42" size="1.27" layer="97" rot="R90">mess with these resistors
-if LEDs are too dim</text>
 <text x="102.87" y="-252.476" size="1.6764" layer="96">0.25W</text>
 <text x="35.56" y="-469.646" size="1.016" layer="97">theoretically handles 8S

Commit message: lite design order
Parts:
- C1, C5: JLC-DNP 2 -> (none)
- LED1: PARTNUM (none) -> LTST-S220KRKT
Changed lines of the file:
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@@
 <grid distance="0.1" unitdist="inch" unit="inch" style="lines" multiple="1" display="no" altdistance="0.01" altunitdist="inch" altunit="inch"/>
 <layers>
-<layer number="1" name="Top" color="4" fill="1" visible="yes" active="no"/>
-<layer number="2" name="Route2" color="1" fill="3" visible="yes" active="no"/>
-<layer number="3" name="Route3" color="4" fill="3" visible="yes" active="no"/>
-<layer number="4" name="Route4" color="1" fill="4" visible="yes" active="no"/>
-<layer number="5" name="Route5" color="4" fill="4" visible="yes" active="no"/>
-<layer number="6" name="Route6" color="1" fill="8" visible="yes" active="no"/>
-<layer number="7" name="Route7" color="4" fill="8" visible="yes" active="no"/>
-<layer number="8" name="Route8" color="1" fill="2" visible="yes" active="no"/>
-<layer number="9" name="Route9" color="4" fill="2" visible="yes" active="no"/>
-<layer number="10" name="Route10" color="1" fill="7" visible="yes" active="no"/>
-<layer number="11" name="Route11" color="4" fill="7" visible="yes" active="no"/>
-<layer number="12" name="Route12" color="1" fill="5" visible="yes" active="no"/>
-<layer number="13" name="Route13" color="4" fill="5" visible="yes" active="no"/>
-<layer number="14" name="Route14" color="1" fill="6" visible="yes" active="no"/>
-<layer number="15" name="Route15" color="4" fill="6" visible="yes" active="no"/>
-<layer number="16" name="Bottom" color="1" fill="1" visible="yes" active="no"/>
-<layer number="17" name="Pads" color="2" fill="1" visible="yes" active="no"/>
-<layer number="18" name="Vias" color="2" fill="1" visible="yes" active="no"/>
-<layer number="19" name="Unrouted" color="6" fill="1" visible="yes" active="no"/>
-<layer number="20" name="Dimension" color="15" fill="1" visible="yes" active="no"/>
-<layer number="21" name="tPlace" color="7" fill="1" visible="yes" active="no"/>
-<layer number="22" name="bPlace" color="7" fill="1" visible="yes" active="no"/>
-<layer number="23" name="tOrigins" color="15" fill="1" visible="yes" active="no"/>
-<layer number="24" name="bOrigins" color="15" fill="1" visible="yes" active="no"/>
-<layer number="25" name="tNames" color="7" fill="1" visible="yes" active="no"/>
-<layer number="26" name="bNames" color="7" fill="1" visible="yes" active="no"/>
-<layer number="27" name="tValues" color="7" fill="1" visible="yes" active="no"/>
-<layer number="28" name="bValues" color="7" fill="1" visible="yes" active="no"/>
+<layer number="1" name="Top" color="4" fill="1" visible="no" active="no"/>
+<layer number="2" name="Route2" color="1" fill="3" visible="no" active="no"/>
+<layer number="3" name="Route3" color="4" fill="3" visible="no" active="no"/>
+<layer number="4" name="Route4" color="1" fill="4" visible="no" active="no"/>
+<layer number="5" name="Route5" color="4" fill="4" visible="no" active="no"/>
+<layer number="6" name="Route6" color="1" fill="8" visible="no" active="no"/>
+<layer number="7" name="Route7" color="4" fill="8" visible="no" active="no"/>
+<layer number="8" name="Route8" color="1" fill="2" visible="no" active="no"/>
+<layer number="9" name="Route9" color="4" fill="2" visible="no" active="no"/>
+<layer number="10" name="Route10" color="1" fill="7" visible="no" active="no"/>
+<layer number="11" name="Route11" color="4" fill="7" visible="no" active="no"/>
+<layer number="12" name="Route12" color="1" fill="5" visible="no" active="no"/>
+<layer number="13" name="Route13" color="4" fill="5" visible="no" active="no"/>
+<layer number="14" name="Route14" color="1" fill="6" visible="no" active="no"/>
+<layer number="15" name="Route15" color="4" fill="6" visible="no" active="no"/>
+<layer number="16" name="Bottom" color="1" fill="1" visible="no" active="no"/>
+<layer number="17" name="Pads" color="2" fill="1" visible="no" active="no"/>
+<layer number="18" name="Vias" color="2" fill="1" visible="no" active="no"/>
+<layer number="19" name="Unrouted" color="6" fill="1" visible="no" active="no"/>
+<layer number="20" name="Dimension" color="15" fill="1" visible="no" active="no"/>
+<layer number="21" name="tPlace" color="7" fill="1" visible="no" active="no"/>
+<layer number="22" name="bPlace" color="7" fill="1" visible="no" active="no"/>
+<layer number="23" name="tOrigins" color="15" fill="1" visible="no" active="no"/>
+<layer number="24" name="bOrigins" color="15" fill="1" visible="no" active="no"/>
+<layer number="25" name="tNames" color="7" fill="1" visible="no" active="no"/>
+<layer number="26" name="bNames" color="7" fill="1" visible="no" active="no"/>
+<layer number="27" name="tValues" color="7" fill="1" visible="no" active="no"/>
+<layer number="28" name="bValues" color="7" fill="1" visible="no" active="no"/>
 <layer number="29" name="tStop" color="7" fill="3" visible="no" active="no"/>
 <layer number="30" name="bStop" color="7" fill="6" visible="no" active="no"/>
@@
 <layer number="35" name="tGlue" color="7" fill="4" visible="no" active="no"/>
 <layer number="36" name="bGlue" color="7" fill="5" visible="no" active="no"/>
-<layer number="37" name="tTest" color="7" fill="1" visible="yes" active="no"/>
-<layer number="38" name="bTest" color="7" fill="1" visible="yes" active="no"/>
+<layer number="37" name="tTest" color="7" fill="1" visible="no" active="no"/>
+<layer number="38" name="bTest" color="7" fill="1" visible="no" active="no"/>
 <layer number="39" name="tKeepout" color="4" fill="11" visible="no" active="no"/>
 <layer number="40" name="bKeepout" color="1" fill="11" visible="no" active="no"/>
@@
 <layer number="44" name="Drills" color="7" fill="1" visible="no" active="no"/>
 <layer number="45" name="Holes" color="7" fill="1" visible="no" active="no"/>
-<layer number="46" name="Milling" color="3" fill="1" visible="yes" active="no"/>
-<layer number="47" name="Measures" color="7" fill="1" visible="yes" active="no"/>
-<layer number="48" name="Document" color="7" fill="1" visible="yes" active="no"/>
-<layer number="49" name="Reference" color="7" fill="1" visible="yes" active="no"/>
-<layer number="50" name="dxf" color="7" fill="1" visible="yes" active="no"/>
-<layer number="51" name="tDocu" color="7" fill="1" visible="yes" active="no"/>
-<layer number="52" name="bDocu" color="7" fill="1" visible="yes" active="no"/>
-<layer number="53" name="tGND_GNDA" color="7" fill="9" visible="yes" active="no"/>
-<layer number="54" name="bGND_GNDA" color="1" fill="9" visible="yes" active="no"/>
-<layer number="56" name="wert" color="7" fill="1" visible="yes" active="no"/>
+<layer number="46" name="Milling" color="3" fill="1" visible="no" active="no"/>
+<layer number="47" name="Measures" color="7" fill="1" visible="no" active="no"/>
+<layer number="48" name="Document" color="7" fill="1" visible="no" active="no"/>
+<layer number="49" name="Reference" color="7" fill="1" visible="no" active="no"/>
+<layer number="50" name="dxf" color="7" fill="1" visible="no" active="no"/>
+<layer number="51" name="tDocu" color="7" fill="1" visible="no" active="no"/>
+<layer number="52" name="bDocu" color="7" fill="1" visible="no" active="no"/>
+<layer number="53" name="tGND_GNDA" color="7" fill="9" visible="no" active="no"/>
+<layer number="54" name="bGND_GNDA" color="1" fill="9" visible="no" active="no"/>
+<layer number="56" name="wert" color="7" fill="1" visible="no" active="no"/>
 <layer number="90" name="Modules" color="5" fill="1" visible="yes" active="yes"/>
 <layer number="91" name="Nets" color="2" fill="1" visible="yes" active="yes"/>
@@
 <part name="LED1" library="hot-wand" deviceset="LED" device="-LTST-S220KRKT" value="LED">
 <attribute name="JLCPARTNUM" value="C284935"/>
+<attribute name="PARTNUM" value="LTST-S220KRKT"/>
 </part>
 <part name="R5" library="hot-wand" deviceset="RESISTOR" device="0603-RES" value="470Ω">
@@
 <part name="SUPPLY2" library="hot-wand" deviceset="24V" device=""/>
 <part name="C1" library="hot-wand" deviceset="CAP" device="1206" value="15n">
-<attribute name="JLC-DNP" value="2"/>
 <attribute name="JLCPARTNUM" value="C3858208"/>
 <attribute name="PARTNUM" value="C3216C0G2E153J160AA"/>
@@
 </part>
 <part name="C5" library="hot-wand" deviceset="CAP" device="1206" value="15n">
-<attribute name="JLC-DNP" value="2"/>
 <attribute name="JLCPARTNUM" value="C3858208"/>
 <attribute name="PARTNUM" value="C3216C0G2E153J160AA"/>
@@
 <attribute name="NAME" x="173.736" y="-332.232" size="1.778" layer="95" rot="R90"/>
 <attribute name="JLCPARTNUM" x="170.18" y="-327.66" size="1.27" layer="96" display="off"/>
+<attribute name="PARTNUM" x="170.18" y="-327.66" size="1.778" layer="96" display="off"/>
 </instance>
 <instance part="R5" gate="G$1" x="170.18" y="-317.5" smashed="yes" rot="R270">

Commit message: filling in part nums
Parts:
- C12, C13: PARTNUM (none) -> UHW1H471MPD
- F1: PARTNUM (none) -> 3518P
- FAN1: PARTNUM (none) -> 0470531000
- IC1: PARTNUM (none) -> R-78K12-2.0
- JP2: PARTNUM (none) -> UJC-H-G-SMT-P6-TR
- JP3: PARTNUM (none) -> XT30PW-M
- Q2, Q3, Q5: PARTNUM (none) -> SIS862ADN-T1-GE3
- Q4: PARTNUM (none) -> DMTH64M2LPDWQ-13
Changed lines of the file:
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@@
 <part name="IC1" library="hot-wand" deviceset="V_REG_78XX" device="-BUCK" value="12V R-78K12-2.0">
 <attribute name="JLC-DNP" value="1"/>
+<attribute name="PARTNUM" value="R-78K12-2.0"/>
 </part>
 <part name="GND21" library="hot-wand" deviceset="GND" device=""/>
@@
 <part name="JP3" library="hot-wand" deviceset="XT-CONNECTOR" device="-XT30PW">
 <attribute name="JLC-DNP" value="1"/>
+<attribute name="PARTNUM" value="XT30PW-M"/>
 </part>
 <part name="GND23" library="hot-wand" deviceset="GND" device=""/>
@@
 <part name="Q2" library="hot-wand" deviceset="MOSFET-NCHANNEL" device="-POWERPAK1212-8" value="SIS862ADN-T1-GE3">
 <attribute name="JLC-DNP" value="1"/>
+<attribute name="PARTNUM" value="SIS862ADN-T1-GE3"/>
 </part>
 <part name="C21" library="hot-wand" deviceset="CAP" device="0603-CAP" value="100n">
@@
 <part name="JP2" library="hot-wand" deviceset="USBC-CHGONLY-4M" device="-DRILL" value="USBC-CHGONLY-4M-DRILL">
 <attribute name="JLC-DNP" value="1"/>
+<attribute name="PARTNUM" value="UJC-H-G-SMT-P6-TR"/>
 </part>
 <part name="Q6" library="hot-wand" deviceset="MOSFET-NCHANNEL" device="SMD" value="2N7002K">
@@
 <part name="Q4" library="hot-wand" deviceset="MOSFET-NCHAN-X2" device="-PPSO8X2" value="DMTH64M2LPDWQ-13">
 <attribute name="JLC-DNP" value="1"/>
+<attribute name="PARTNUM" value="DMTH64M2LPDWQ-13"/>
 </part>
 <part name="R9" library="hot-wand" deviceset="RESISTOR" device="0603-RES" value="4K3">
@@
 <part name="F1" library="hot-wand" deviceset="FUSE" device="X20MM">
 <attribute name="JLC-DNP" value="1"/>
+<attribute name="PARTNUM" value="3518P"/>
 </part>
 <part name="GND2" library="hot-wand" deviceset="GND" device=""/>
@@
 <part name="C12" library="hot-wand" deviceset="CAP_POL" device="PTH5" value="470u">
 <attribute name="JLC-DNP" value="1"/>
+<attribute name="PARTNUM" value="UHW1H471MPD"/>
 </part>
 <part name="GND7" library="hot-wand" deviceset="GND" device=""/>
@@
 <part name="C13" library="hot-wand" deviceset="CAP_POL" device="PTH4" value="470u">
 <attribute name="JLC-DNP" value="1"/>
+<attribute name="PARTNUM" value="UHW1H471MPD"/>
 </part>
 <part name="R16" library="hot-wand" deviceset="RESISTOR" device="0603-RES" value="1K">
@@
 <part name="Q5" library="hot-wand" deviceset="MOSFET-NCHANNEL" device="-POWERPAK1212-8" value="SIS862ADN-T1-GE3">
 <attribute name="JLC-DNP" value="1"/>
+<attribute name="PARTNUM" value="SIS862ADN-T1-GE3"/>
 </part>
 <part name="JP4" library="hot-wand" deviceset="M02" device="PTH3">
@@
 </part>
 <part name="GND38" library="hot-wand" deviceset="GND" device=""/>
-<part name="FAN1" library="hot-wand" deviceset="FAN-CONN-X4" device="-CONN-X4"/>
+<part name="FAN1" library="hot-wand" deviceset="FAN-CONN-X4" device="-CONN-X4">
+<attribute name="PARTNUM" value="0470531000"/>
+</part>
 <part name="SJ6" library="hot-wand" deviceset="SOLDERJUMPER_2WAY" device="S"/>
 <part name="SJ7" library="hot-wand" deviceset="SOLDERJUMPER_2WAY" device="S"/>
@@
 <part name="Q3" library="hot-wand" deviceset="MOSFET-NCHANNEL" device="-POWERPAK1212-8" value="SIS862ADN-T1-GE3">
 <attribute name="JLC-DNP" value="1"/>
+<attribute name="PARTNUM" value="SIS862ADN-T1-GE3"/>
 </part>
 <part name="R30" library="hot-wand" deviceset="RESISTOR" device="0805-RES" value="100Ω">

Commit message: renumbered component names
Parts:
- removed R33: 22K, hot-wand:RESISTOR0603-RES
- added R12: 22K, hot-wand:RESISTOR0603-RES
- R29: value 22K -> 100Ω; device hot-wand:RESISTOR0603-RES -> hot-wand:RESISTOR0805-RES; JLCPARTNUM C31850 -> C441975
- R30: value 100Ω -> 56K; device hot-wand:RESISTOR0805-RES -> hot-wand:RESISTOR0603-RES; JLCPARTNUM C441975 -> C23206
- R31: value 56K -> 2K; JLCPARTNUM C23206 -> C22975
- R32: value 2K -> 22K; JLCPARTNUM C22975 -> C31850
Connections:
- net GND: now also R31.2; no longer R33.2
- net N$32: now also R12.1; no longer R29.1
- net N$43: now also R29.2; no longer R30.2
- net N$66: now also R29.1; no longer R30.1
- net N$68: now also R30.2; no longer R31.2
- net N$71: now also R30.1; no longer R33.1
- net VCD: now also R12.2; no longer R29.2
Other:
- moved on the sheet: R29, R30, R31, R32
Changed lines of the file:
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@@
 </part>
 <part name="GND40" library="hot-wand" deviceset="GND" device=""/>
-<part name="R29" library="hot-wand" deviceset="RESISTOR" device="0603-RES" value="22K">
+<part name="R12" library="hot-wand" deviceset="RESISTOR" device="0603-RES" value="22K">
 <attribute name="JLCPARTNUM" value="C31850"/>
 </part>
@@
 <attribute name="PARTNUM" value="SIS862ADN-T1-GE3"/>
 </part>
-<part name="R30" library="hot-wand" deviceset="RESISTOR" device="0805-RES" value="100Ω">
+<part name="R29" library="hot-wand" deviceset="RESISTOR" device="0805-RES" value="100Ω">
 <attribute name="JLCPARTNUM" value="C441975"/>
 </part>
@@
 <attribute name="JLCPARTNUM" value="C14663"/>
 </part>
-<part name="R31" library="hot-wand" deviceset="RESISTOR" device="0603-RES" value="56K">
+<part name="R30" library="hot-wand" deviceset="RESISTOR" device="0603-RES" value="56K">
 <attribute name="JLCPARTNUM" value="C23206"/>
 </part>
@@
 <attribute name="JLCPARTNUM" value="C14663"/>
 </part>
-<part name="R33" library="hot-wand" deviceset="RESISTOR" device="0603-RES" value="22K">
+<part name="R32" library="hot-wand" deviceset="RESISTOR" device="0603-RES" value="22K">
 <attribute name="JLCPARTNUM" value="C31850"/>
 </part>
-<part name="R32" library="hot-wand" deviceset="RESISTOR" device="0603-RES" value="2K">
+<part name="R31" library="hot-wand" deviceset="RESISTOR" device="0603-RES" value="2K">
 <attribute name="JLCPARTNUM" value="C22975"/>
 </part>
@@
 </instance>
 <instance part="GND40" gate="1" x="27.94" y="-203.2"/>
-<instance part="R29" gate="G$1" x="76.2" y="-513.08" smashed="yes" rot="R90">
+<instance part="R12" gate="G$1" x="76.2" y="-513.08" smashed="yes" rot="R90">
 <attribute name="NAME" x="79.7814" y="-516.89" size="1.778" layer="95" rot="R90"/>
 <attribute name="VALUE" x="80.518" y="-511.81" size="1.778" layer="96" rot="R270"/>
@@
 <attribute name="JLC-DNP" x="121.92" y="-477.52" size="1.778" layer="96" rot="R90" display="off"/>
 </instance>
-<instance part="R30" gate="G$1" x="129.54" y="-487.68">
+<instance part="R29" gate="G$1" x="129.54" y="-487.68">
 <attribute name="JLCPARTNUM" x="129.54" y="-487.68" size="1.778" layer="96" display="off"/>
 </instance>
@@
 <attribute name="VALUE" x="144.272" y="-490.347" size="1.778" layer="96" rot="R180"/>
 </instance>
-<instance part="R31" gate="G$1" x="139.7" y="-508" smashed="yes" rot="R180">
+<instance part="R30" gate="G$1" x="139.7" y="-508" smashed="yes" rot="R180">
 <attribute name="NAME" x="143.51" y="-504.4186" size="1.778" layer="95" rot="R180"/>
 <attribute name="VALUE" x="143.51" y="-502.158" size="1.778" layer="96" rot="R180"/>
@@
 <attribute name="VALUE" x="154.432" y="-490.347" size="1.778" layer="96" rot="R180"/>
 </instance>
-<instance part="R33" gate="G$1" x="154.94" y="-520.7" smashed="yes">
+<instance part="R32" gate="G$1" x="154.94" y="-520.7" smashed="yes">
 <attribute name="NAME" x="151.13" y="-524.2814" size="1.778" layer="95"/>
 <attribute name="VALUE" x="156.21" y="-525.018" size="1.778" layer="96" rot="R180"/>
 </instance>
-<instance part="R32" gate="G$1" x="154.94" y="-513.08" smashed="yes">
+<instance part="R31" gate="G$1" x="154.94" y="-513.08" smashed="yes">
 <attribute name="NAME" x="151.13" y="-516.6614" size="1.778" layer="95"/>
 <attribute name="VALUE" x="151.13" y="-511.556" size="1.778" layer="96"/>
@@
 </segment>
 <segment>
-<pinref part="R32" gate="G$1" pin="2"/>
+<pinref part="R31" gate="G$1" pin="2"/>
 <pinref part="GND44" gate="1" pin="GND"/>
 <wire x1="160.02" y1="-513.08" x2="162.56" y2="-513.08" width="0.1524" layer="91"/>
 <wire x1="162.56" y1="-513.08" x2="162.56" y2="-520.7" width="0.1524" layer="91"/>
-<pinref part="R33" gate="G$1" pin="2"/>
+<pinref part="R32" gate="G$1" pin="2"/>
 <wire x1="162.56" y1="-520.7" x2="162.56" y2="-523.24" width="0.1524" layer="91"/>
 <wire x1="160.02" y1="-520.7" x2="162.56" y2="-520.7" width="0.1524" layer="91"/>
@@
 </segment>
 <segment>
-<pinref part="R29" gate="G$1" pin="2"/>
+<pinref part="R12" gate="G$1" pin="2"/>
 <wire x1="76.2" y1="-508" x2="76.2" y2="-505.46" width="0.1524" layer="91"/>
 <label x="76.2" y="-505.46" size="1.016" layer="95" rot="R90" xref="yes"/>
@@
 <pinref part="U3" gate="A" pin="EN_UVLO"/>
 <wire x1="45.72" y1="-520.7" x2="76.2" y2="-520.7" width="0.1524" layer="91"/>
-<pinref part="R29" gate="G$1" pin="1"/>
+<pinref part="R12" gate="G$1" pin="1"/>
 <wire x1="76.2" y1="-520.7" x2="86.36" y2="-520.7" width="0.1524" layer="91"/>
 <wire x1="76.2" y1="-518.16" x2="76.2" y2="-520.7" width="0.1524" layer="91"/>
@@
 <pinref part="Q3" gate="G$1" pin="G"/>
 <wire x1="121.92" y1="-487.68" x2="121.92" y2="-485.14" width="0.1524" layer="91"/>
-<pinref part="R30" gate="G$1" pin="1"/>
+<pinref part="R29" gate="G$1" pin="1"/>
 <wire x1="124.46" y1="-487.68" x2="121.92" y2="-487.68" width="0.1524" layer="91"/>
 <junction x="121.92" y="-487.68"/>
@@
 <segment>
 <pinref part="U3" gate="A" pin="SW"/>
-<pinref part="R31" gate="G$1" pin="2"/>
+<pinref part="R30" gate="G$1" pin="2"/>
 <wire x1="132.08" y1="-508" x2="134.62" y2="-508" width="0.1524" layer="91"/>
 </segment>
@@
 <net name="N$71" class="0">
 <segment>
-<pinref part="R31" gate="G$1" pin="1"/>
+<pinref part="R30" gate="G$1" pin="1"/>
 <wire x1="144.78" y1="-508" x2="147.32" y2="-508" width="0.1524" layer="91"/>
 <wire x1="147.32" y1="-508" x2="147.32" y2="-513.08" width="0.1524" layer="91"/>
-<pinref part="R32" gate="G$1" pin="1"/>
+<pinref part="R31" gate="G$1" pin="1"/>
 <wire x1="147.32" y1="-513.08" x2="149.86" y2="-513.08" width="0.1524" layer="91"/>
 <pinref part="U3" gate="A" pin="OV"/>
 <wire x1="132.08" y1="-513.08" x2="147.32" y2="-513.08" width="0.1524" layer="91"/>
 <junction x="147.32" y="-513.08"/>
-<pinref part="R33" gate="G$1" pin="1"/>
+<pinref part="R32" gate="G$1" pin="1"/>
 <wire x1="149.86" y1="-520.7" x2="147.32" y2="-520.7" width="0.1524" layer="91"/>
 <wire x1="147.32" y1="-520.7" x2="147.32" y2="-513.08" width="0.1524" layer="91"/>
@@
 <net name="N$43" class="0">
 <segment>
-<pinref part="R30" gate="G$1" pin="2"/>
+<pinref part="R29" gate="G$1" pin="2"/>
 <pinref part="C25" gate="G$1" pin="2"/>
 <wire x1="134.62" y1="-487.68" x2="137.16" y2="-487.68" width="0.1524" layer="91"/>

Commit message: out of stock part number options
Parts:
- C6: JLCPARTNUM C2261646 -> C2261646;C2170837;C2175075; PARTNUM GRM31B5C2E103JWA1L -> C3216C0G2E103J115AA
Changed lines of the file:
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@@
 </part>
 <part name="C6" library="hot-wand" deviceset="CAP" device="1206" value="10n">
-<attribute name="JLCPARTNUM" value="C2261646"/>
-<attribute name="PARTNUM" value="GRM31B5C2E103JWA1L"/>
+<attribute name="JLCPARTNUM" value="C2261646;C2170837;C2175075"/>
+<attribute name="PARTNUM" value="C3216C0G2E103J115AA"/>
 </part>
 <part name="C7" library="hot-wand" deviceset="CAP" device="1206" value="10n">

Commit message: new part number for small mosfet to lower costs
Parts:
- Q6: JLCPARTNUM C5224211;C54347659 -> C14498;C547263;C5224211;C54347659; PARTNUM 2N7002K;SSM3K388R,LF -> 2N7002K;SSM3K388R,LF;Si2318CDS-T1-GE3;PMV60ENEAR
- Q7: JLCPARTNUM C96615 -> C14498;C547263;C96615; PARTNUM G3404;MMFTN3404A;PJA3404A -> G3404;MMFTN3404A;PJA3404A;Si2318CDS-T1-GE3;PMV60ENEAR
Changed lines of the file:
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@@
 </part>
 <part name="Q6" library="hot-wand" deviceset="MOSFET-NCHANNEL" device="SMD" value="2N7002K">
-<attribute name="JLCPARTNUM" value="C5224211;C54347659"/>
-<attribute name="PARTNUM" value="2N7002K;SSM3K388R,LF"/>
+<attribute name="JLCPARTNUM" value="C14498;C547263;C5224211;C54347659"/>
+<attribute name="PARTNUM" value="2N7002K;SSM3K388R,LF;Si2318CDS-T1-GE3;PMV60ENEAR"/>
 </part>
 <part name="GND28" library="hot-wand" deviceset="GND" device=""/>
@@
 </part>
 <part name="Q7" library="hot-wand" deviceset="MOSFET-NCHANNEL" device="SMD" value="G3404">
-<attribute name="JLCPARTNUM" value="C96615"/>
-<attribute name="PARTNUM" value="G3404;MMFTN3404A;PJA3404A"/>
+<attribute name="JLCPARTNUM" value="C14498;C547263;C96615"/>
+<attribute name="PARTNUM" value="G3404;MMFTN3404A;PJA3404A;Si2318CDS-T1-GE3;PMV60ENEAR"/>
 </part>
 <part name="R27" library="hot-wand" deviceset="RESISTOR" device="0603-RES" value="470Ω">
